Commit message: Added mimic joint and such

File: robotiq_2f_85_gripper_visualization/urdf/robotiq_arg2f_85.gazebo.xacro (robot description, xacro)
@@ -1,39 +1,45 @@
 <?xml version="1.0"?>
-<robot xmlns:xacro="http://wiki.ros.org/xacro">
-    <xacro:macro name="robotiq_arg2f_gazebo" params="prefix">
+<robot xmlns:xacro="http://ros.org/wiki/xacro">
+  <xacro:macro name="robotiq_arg2f_85_gazebo" params="prefix">
     <!-- To fix broken gripper in gazebo according to the following issue-->
     <!--https://github.com/ros-industrial/robotiq/issues/150-->
-        <gazebo>
-            <plugin filename="libgazebo_utils_mimic_joint_plugin.so" name="${prefix}mimic_robotiq_140_1">
+    <gazebo>
+             <!-- loading plugin: mimic joints works in gazebo now-->
+             <plugin filename="librobotiq_gazebo_mimic_joint_plugin.so" name="${prefix}mimic_robotiq_85_4">
                 <joint>${prefix}finger_joint</joint>
                 <mimicJoint>${prefix}right_outer_knuckle_joint</mimicJoint>
+                <multiplier>1.0</multiplier>
+                <!--<multiplier>-1.0</multiplier>-->
+                <!--<offset>0.0</offset>-->
+            </plugin>
+            <plugin filename="librobotiq_gazebo_mimic_joint_plugin.so" name="${prefix}mimic_robotiq_85_2">
+                <joint>${prefix}finger_joint</joint>
+                <mimicJoint>${prefix}left_inner_finger_joint</mimicJoint>
                 <multiplier>-1.0</multiplier>
-                <offset>0.0</offset>
+                <!--<multiplier>1.0</multiplier>-->
+                <!--<offset>0.0</offset>-->
             </plugin>
-            <plugin filename="libgazebo_utils_mimic_joint_plugin.so" name="${prefix}mimic_robotiq_140_2">
+            <plugin filename="librobotiq_gazebo_mimic_joint_plugin.so" name="${prefix}mimic_robotiq_85_6">
+                <joint>${prefix}finger_joint</joint>
+                <mimicJoint>${prefix}right_inner_finger_joint</mimicJoint>
+                <multiplier>-1.0</multiplier>
+                <!--<multiplier>1.0</multiplier>-->
+                <!--<offset>0.0</offset>-->
+            </plugin>
+            <plugin filename="librobotiq_gazebo_mimic_joint_plugin.so" name="${prefix}mimic_robotiq_85_3">
                 <joint>${prefix}finger_joint</joint>
                 <mimicJoint>${prefix}left_inner_knuckle_joint</mimicJoint>
-                <multiplier>-1.0</multiplier>
-                <offset>0.0</offset>
+                <multiplier>1.0</multiplier>
+                <!--<multiplier>-1.0</multiplier>-->
+                <!--<offset>0.0</offset>-->
             </plugin>
-            <plugin filename="libgazebo_utils_mimic_joint_plugin.so" name="${prefix}mimic_robotiq_140_3">
+            <plugin filename="librobotiq_gazebo_mimic_joint_plugin.so" name="${prefix}mimic_robotiq_85_5">
                 <joint>${prefix}finger_joint</joint>
                 <mimicJoint>${prefix}right_inner_knuckle_joint</mimicJoint>
-                <multiplier>-1.0</multiplier>
-                <offset>0.0</offset>
-            </plugin>
-            <plugin filename="libgazebo_utils_mimic_joint_plugin.so" name="${prefix}mimic_robotiq_140_4">
-                <joint>${prefix}finger_joint</joint>
-                <mimicJoint>${prefix}left_inner_finger_joint</mimicJoint>
                 <multiplier>1.0</multiplier>
-                <offset>0.0</offset>
-            </plugin>
-            <plugin filename="libgazebo_utils_mimic_joint_plugin.so" name="${prefix}mimic_robotiq_140_5">
-                <joint>${prefix}finger_joint</joint>
-                <mimicJoint>${prefix}right_inner_finger_joint</mimicJoint>
-                <multiplier>1.0</multiplier>
-                <offset>0.0</offset>
+                <!--<multiplier>-1.0</multiplier>-->
+                <!--<offset>0.0</offset>-->
             </plugin>
         </gazebo>
-    </xacro:macro>
+  </xacro:macro>
 </robot>

File: robotiq_2f_85_gripper_visualization/urdf/robotiq_arg2f_85_model_macro.xacro (robot description, xacro)
@@ -2,4 +2,5 @@
 <robot xmlns:xacro="http://ros.org/wiki/xacro">
   <xacro:include filename="$(find robotiq_2f_85_gripper_visualization)/urdf/robotiq_arg2f_transmission.xacro" />
+  <xacro:include filename="$(find robotiq_2f_85_gripper_visualization)/urdf/robotiq_arg2f_85.gazebo.xacro"/>
   <xacro:macro name="outer_knuckle" params="prefix fingerprefix stroke">
     <link name="${prefix}${fingerprefix}_outer_knuckle">
@@ -188,4 +189,5 @@
     <xacro:right_outer_knuckle_joint prefix="${prefix}"/>
     <xacro:robotiq_arg2f_transmission prefix="${prefix}"/>
+    <xacro:robotiq_arg2f_85_gazebo prefix="${prefix}"/>
   </xacro:macro>
 </robot>

File: robotiq_2f_85_gripper_visualization/urdf/robotiq_arg2f_transmission.xacro (robot description, xacro)
@@ -5,5 +5,5 @@
       <type>transmission_interface/SimpleTransmission</type>
       <joint name="${prefix}finger_joint">
-        <hardwareInterface>hardware_interface/PositionJointInterface</hardwareInterface> <!-- EffortJointInterface-->
+        <hardwareInterface>hardware_interface/EffortJointInterface</hardwareInterface>
         <!--<hardwareInterface>hardware_interface/PositionJointInterface</hardwareInterface>-->
       </joint>
