Commit message: Add damping and friction to finger, now works in gazebo

File: robotiq_2f_85_gripper_visualization/urdf/robotiq_arg2f_85_model_macro.xacro (robot description, xacro)
@@ -3,4 +3,6 @@
   <xacro:include filename="$(find robotiq_2f_85_gripper_visualization)/urdf/robotiq_arg2f_transmission.xacro" />
   <xacro:include filename="$(find robotiq_2f_85_gripper_visualization)/urdf/robotiq_arg2f_85.gazebo.xacro"/>
+  <xacro:property name="finger_joint_damping" value="0.0025"/>
+  <xacro:property name="finger_joint_friction" value="0.0"/>
   <xacro:macro name="outer_knuckle" params="prefix fingerprefix stroke">
     <link name="${prefix}${fingerprefix}_outer_knuckle">
@@ -137,5 +139,5 @@
       <child link="${prefix}${fingerprefix}_inner_knuckle" />
       <axis xyz="1 0 0" />
-      <limit lower="0" upper="0.8757" velocity="2.0" effort="1000" />
+      <limit lower="0" upper="0.8757" velocity="0.5" effort="1000" />
       <mimic joint="${prefix}finger_joint" multiplier="1" offset="0" />
     </joint>
@@ -147,5 +149,5 @@
       <child link="${prefix}${fingerprefix}_inner_finger" />
       <axis xyz="1 0 0" />
-      <limit lower="0" upper="0.8757" velocity="2.0" effort="1000" />
+      <limit lower="-0.8757" upper="0.0" velocity="0.5" effort="1000" />
       <mimic joint="${prefix}finger_joint" multiplier="-1" offset="0" />
     </joint>
@@ -166,5 +168,6 @@
       <child link="${prefix}left_outer_knuckle" />
       <axis xyz="1 0 0" />
-      <limit lower="0" upper="0.8" velocity="2.0" effort="1000" />
+      <limit lower="0" upper="0.8" velocity="0.5" effort="1000" />
+      <dynamics damping="${finger_joint_damping}" friction="${finger_joint_friction}"/>
     </joint>
     <xacro:finger_joints prefix="${prefix}" fingerprefix="left" reflect="1.0"/>
@@ -176,5 +179,5 @@
       <child link="${prefix}right_outer_knuckle" />
       <axis xyz="1 0 0" />
-      <limit lower="0" upper="0.81" velocity="2.0" effort="1000" />
+      <limit lower="0" upper="0.81" velocity="0.5" effort="1000" />
       <mimic joint="${prefix}finger_joint" multiplier="1" offset="0" />
     </joint>
